File: schematics/kiCad/blinky-cube.kicad_pcb (KiCad board)
At the start: 2 copper layers, 86.6 x 49.7 mm, 26 parts, among them J1 Screw_Terminal_01x03, J2 Screw_Terminal_01x03, J3 Screw_Terminal_01x03, SW1 SW_Push, U1 Pico, U2 LM4040LP-3

Commit message: first commit
Parts:
- removed C2, C3, C4, C5, C6: 1uF, Capacitor_SMD:C_1206_3216Metric_Pad1.33x1.80mm_HandSolder
- removed R10, R12, R8: 120k, Resistor_SMD:R_1206_3216Metric_Pad1.30x1.75mm_HandSolder
- removed R11, R7, R9: 82k, Resistor_SMD:R_1206_3216Metric_Pad1.30x1.75mm_HandSolder
- removed R3: 220, Resistor_SMD:R_1206_3216Metric_Pad1.30x1.75mm_HandSolder
- removed R4, R5, R6: 100k, Resistor_SMD:R_1206_3216Metric_Pad1.30x1.75mm_HandSolder
- added U3: MAX31865, MAX31865:MAX31865, F.Cu at (138.7, 107.8)
- C1: footprint Capacitor_SMD:C_1206_3216Metric_Pad1.33x1.80mm_HandSolder -> Capacitor_THT:C_Disc_D4.3mm_W1.9mm_P5.00mm; moved to F.Cu
- J1, J2: value Screw_Terminal_01x03 -> Screw_Terminal_01x04; footprint TerminalBlock:TerminalBlock_bornier-3_P5.08mm -> TerminalBlock:TerminalBlock_bornier-4_P5.08mm
- J3: value Screw_Terminal_01x03 -> Screw_Terminal_01x02; footprint TerminalBlock:TerminalBlock_bornier-3_P5.08mm -> TerminalBlock:TerminalBlock_bornier-2_P5.08mm
- R1, R2: footprint Resistor_SMD:R_1206_3216Metric_Pad1.30x1.75mm_HandSolder -> Resistor_THT:R_Axial_DIN0207_L6.3mm_D2.5mm_P7.62mm_Horizontal; moved to F.Cu
- U2: value LM4040LP-3 -> MAX31865; footprint Package_TO_SOT_THT:TO-92_Inline -> MAX31865:MAX31865
- moved J3 87.1 mm to (181.9, 111.6), turned to 90 degrees
- moved J1 78.7 mm to (105.5, 76.0)
- moved G*** 32.3 mm to (128.6, 83.6)
- moved U2 22.6 mm to (138.6, 77.2), turned to 90 degrees
- moved R2 21.9 mm to (182.0, 81.5), turned to 90 degrees
- moved J2 21.5 mm to (105.5, 106.5), turned to 90 degrees
- moved U1 19.0 mm to (161.0, 83.0), turned to 180 degrees
- moved C1 16.6 mm to (179.2, 98.9), turned to 0 degrees
- moved R1 4.33 mm to (169.1, 53.2)
- moved D1 2.79 mm to (180.6, 55.7), turned to 0 degrees
- moved SW1 1.20 mm to (184.2, 62.6)
Connections:
- D1 pad 2: Net-(D1-Pad2) -> Net-(U1-Pad19)
- J1 pad 1: Net-(C2-Pad2) -> Net-(J1-Pad1)
- J1 pad 2: Net-(C1-Pad1) -> Net-(J1-Pad2)
- J1 pad 3: GND -> Net-(J1-Pad3)
- J2 pad 2: GND -> Net-(J2-Pad2)
- J3 pad 1: GND -> Net-(C1-Pad1)
- J3 pad 2: Net-(C5-Pad1) -> GND
- U1 pad 10: unconnected-(U1-Pad10) -> Net-(R2-Pad1)
- U1 pad 19: unconnected-(U1-Pad19) -> Net-(U1-Pad19)
- U1 pad 20: unconnected-(U1-Pad20) -> Net-(U2-Pad8)
- U1 pad 21: unconnected-(U1-Pad21) -> Net-(U1-Pad21)
- U1 pad 22: unconnected-(U1-Pad22) -> Net-(U1-Pad22)
- U1 pad 23: GND -> unconnected-(U1-Pad23)
- U1 pad 24: unconnected-(U1-Pad24) -> Net-(U1-Pad24)
- U1 pad 25: unconnected-(U1-Pad25) -> Net-(U1-Pad25)
- U1 pad 26: unconnected-(U1-Pad26) -> Net-(U3-Pad8)
- U1 pad 27: unconnected-(U1-Pad27) -> Net-(U3-Pad7)
- U1 pad 31: Net-(R11-Pad2) -> unconnected-(U1-Pad31)
- U1 pad 32: Net-(R10-Pad1) -> unconnected-(U1-Pad32)
- U1 pad 34: Net-(R7-Pad2) -> unconnected-(U1-Pad34)
- U1 pad 35: Net-(R3-Pad2) -> unconnected-(U1-Pad35)
- U1 pad 39: unconnected-(U1-Pad39) -> Net-(C1-Pad1)
- U1 pad 4: Net-(D1-Pad2) -> unconnected-(U1-Pad4)
- U1 pad 40: Net-(C1-Pad1) -> unconnected-(U1-Pad40)
- U1 pad 5: Net-(R2-Pad1) -> unconnected-(U1-Pad5)
- U2 pad 1: (no net) -> Net-(SW1-Pad1)
- U2 pad 2: Net-(R3-Pad2) -> GND
- U2 pad 3: GND -> unconnected-(U2-Pad3)
Routing:
- net Net-(C2-Pad2): track 114.8 -> 0.00 mm, vias 3 -> 0
- net Net-(SW1-Pad1): track 40.4 -> 123.9 mm
- net Net-(U1-Pad21): track 0.00 -> 61.8 mm
- net Net-(R7-Pad2): track 61.1 -> 0.00 mm
- net Net-(R11-Pad2): track 59.4 -> 0.00 mm
- net Net-(U1-Pad24): track 0.00 -> 50.9 mm, vias 0 -> 1
- net Net-(U1-Pad25): track 0.00 -> 49.3 mm
- net Net-(R10-Pad1): track 43.4 -> 0.00 mm
- net Net-(U2-Pad8): track 0.00 -> 34.9 mm
- net Net-(U3-Pad7): track 0.00 -> 29.9 mm
- net Net-(U3-Pad8): track 0.00 -> 29.1 mm
- net Net-(D1-Pad2): track 29.1 -> 0.00 mm
- net Net-(C5-Pad1): track 23.3 -> 0.00 mm
- net Net-(R3-Pad2): track 19.5 -> 0.00 mm
- net Net-(C1-Pad1): track 31.7 -> 51.0 mm
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Other:
- board size 86.6 x 49.7 mm -> 86.6 x 67.4 mm
