File: schematics/kiCad/blinky-cube.kicad_pcb (KiCad board)
At the start: 2 copper layers, 86.6 x 67.4 mm, 12 parts, among them J1 Screw_Terminal_01x04, J2 Screw_Terminal_01x04, J3 Screw_Terminal_01x02, SW1 SW_Push, U1 Pico, U2 MAX31865, U3 MAX31865

Commit message: added logo
Other:
- board text added: "blinky-max31865-v1"
